File: mt6835-hoverboard.kicad_pcb (KiCad board)
At the start: 2 copper layers, 14.2 x 14.2 mm, 10 parts, among them U1 MT6835

Commit message: update schematic
Parts:
- renumbered REF** to J1, REF** to J2, REF** to J3
