File: mt6835-hoverboard.kicad_pcb (KiCad board)
At the start: 2 copper layers, 24 x 32 mm, 14 parts, among them J1 PinHeader_1x06_P1.27mm_Vertic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, J2 PinHeader_1x06_P1.00mm_Vertic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, J3 PinHeader_1x06_P1.00mm_Vertic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, U1 MT6835

Commit message: Revision 1.1: Good for production
Connections:
- REF** pad 1: (no net) -> GND (x4)
Routing:
- net GND: track 2.90 -> 403.7 mm
- net (no net): track 385.7 -> 0.00 mm
Other:
- outline, holes or cut-outs redrawn
- board text added: "mcells, 07.2024"
- board text added: "rev 1.1"
- board text removed: "mcells 07.2024"
- board text removed: "rev 1.0"

Commit message: Rev 1.2: Move pinout silkscreen slightly
Other:
- board text added: "rev 1.2"
- board text removed: "rev 1.1"
Changed lines of the file:
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@@
 		)
 	)
-	(gr_text "rev 1.1"
+	(gr_text "rev 1.2"
 		(at 151.6 96.6 340)
 		(layer "B.SilkS" knockout)
@@
 	)
 	(gr_text "CAL\nW\nV\nU\n+\n-"
-		(at 147.1 92.8 0)
+		(at 147.35 92.8 0)
 		(layer "B.SilkS")
 		(effects
@@
 	)
 	(gr_text "PWM\nZ\nB\nA\n+\n-"
-		(at 152.905 92.8425 0)
+		(at 152.65 92.85 0)
 		(layer "B.SilkS")
 		(effects
